Commit message: Added placer gripper

File: models/hydra/hydra.urdf.xacro (robot description, xacro)
@@ -18,4 +18,7 @@
     <xacro:ur10_robot prefix="placer_" joint_limited="false" />
   </xacro:unless>
+  <!-- Gripper -->
+  <xacro:include filename="$(find hydra)/models/gripper_placer/gripper_placer.urdf.xacro"/>
+  <!-- Attach placer manipulator to world -->
   <link name="world" />
   <joint name="placer_world_joint" type="fixed">
@@ -23,4 +26,10 @@
     <child link = "placer_base_link" />
     <origin xyz="0.0 0.0 0.0" rpy="0.0 0.0 0.0" />
+  </joint>
+  <!-- joint to attach mount for tool to UR10 -->
+  <joint name="mount_gripper_to_placer" type="fixed">
+    <origin xyz="0 0 0" rpy="0 0 0" />
+    <parent link="placer_tool0" />
+    <child link="gripper_center" />
   </joint>
   <!-- UR10 description for attacher robot -->
