Commit message: Changed gripper prismatic axis

File: models/gripper_placer/gripper_placer.urdf.xacro (robot description, xacro)
@@ -19,5 +19,5 @@
   <link name="side_p" >
     <visual>
-      <origin xyz="0 0.04185 0" rpy="0 0 0" />
+      <origin xyz="0 0 0" rpy="0 0 0" />
       <geometry>
 	<mesh filename="package://hydra/models/gripper_placer/meshes/gripper_pad_v2.stl" scale="0.01 0.01 0.01" />
@@ -25,5 +25,5 @@
     </visual>
     <collision>
-      <origin xyz="0 0.04185 0" rpy="0 0 0" />
+      <origin xyz="0 0 0" rpy="0 0 0" />
       <geometry>
 	<mesh filename="package://hydra/models/gripper_placer/meshes/gripper_pad_v2.stl" scale="0.01 0.01 0.01" />
@@ -38,5 +38,5 @@
   <link name="side_d" >
     <visual>
-      <origin xyz="0 -0.04185 0" rpy="0 0 ${pi}" />
+      <origin xyz="0 0 0" rpy="0 0 ${pi}" /><!--origin xyz="0 0.04185 0" rpy="0 0 ${pi}" /-->
       <geometry>
 	<mesh filename="package://hydra/models/gripper_placer/meshes/gripper_pad_v2.stl" scale="0.01 0.01 0.01" />
@@ -44,5 +44,5 @@
     </visual>
     <collision>
-      <origin xyz="0 -0.04185 0" rpy="0 0 ${pi}" />
+      <origin xyz="0 0 0" rpy="0 0 ${pi}" />
       <geometry>
 	<mesh filename="package://hydra/models/gripper_placer/meshes/gripper_pad_v2.stl" scale="0.01 0.01 0.01" />
@@ -57,4 +57,5 @@
   <joint name="gripper_joint_p" type="prismatic">
     <origin xyz="0 0 0" rpy="0 0 0" />
+    <axis xyz="0 1 0" />
     <parent link="gripper_center" />
     <child link="side_p" />
@@ -63,4 +64,5 @@
   <joint name="gripper_joint_d" type="prismatic">
     <origin xyz="0 0 0" rpy="0 0 0" />
+    <axis xyz="0 1 0" />
     <parent link="gripper_center" />
     <child link="side_d" />

Commit message: Updated demo, launch, and world

File: models/gripper_placer/gripper_placer.urdf.xacro (robot description, xacro)
@@ -9,4 +9,6 @@
   <xacro:property name="gripper_min_depth" value="0.001" />  <!-- Default is 0 -->
   <xacro:property name="gripper_max_vel" value="0.01" />  <!-- Default is 0.01 -->
+  <!-- Variable for the scale used when importing STL -->
+  <xacro:property name="stl_scale" value="0.0254" />  <!-- 0.0393701 -->
   <!-- Phantom link for center of gripper -->
   <link name="gripper_center" >
@@ -19,13 +21,13 @@
   <link name="side_p" >
     <visual>
-      <origin xyz="0 0 0" rpy="0 0 0" />
+      <origin xyz="0 0 0.11485" rpy="0 0 0" />
       <geometry>
-	<mesh filename="package://hydra/models/gripper_placer/meshes/gripper_pad_v2.stl" scale="0.01 0.01 0.01" />
+	<mesh filename="package://hydra/models/gripper_placer/meshes/gripper_pad_v2.stl" scale="${stl_scale} ${stl_scale} ${stl_scale}" />
       </geometry>
     </visual>
     <collision>
-      <origin xyz="0 0 0" rpy="0 0 0" />
+      <origin xyz="0 0 0.11485" rpy="0 0 0" />
       <geometry>
-	<mesh filename="package://hydra/models/gripper_placer/meshes/gripper_pad_v2.stl" scale="0.01 0.01 0.01" />
+	<mesh filename="package://hydra/models/gripper_placer/meshes/gripper_pad_v2.stl" scale="${stl_scale} ${stl_scale} ${stl_scale}" />
       </geometry>
     </collision>
@@ -38,13 +40,13 @@
   <link name="side_d" >
     <visual>
-      <origin xyz="0 0 0" rpy="0 0 ${pi}" /><!--origin xyz="0 0.04185 0" rpy="0 0 ${pi}" /-->
+      <origin xyz="0 0 0.11485" rpy="0 0 ${pi}" /><!--origin xyz="0 0.04185 0" rpy="0 0 ${pi}" /-->
       <geometry>
-	<mesh filename="package://hydra/models/gripper_placer/meshes/gripper_pad_v2.stl" scale="0.01 0.01 0.01" />
+	<mesh filename="package://hydra/models/gripper_placer/meshes/gripper_pad_v2.stl" scale="${stl_scale} ${stl_scale} ${stl_scale}" />
       </geometry>
     </visual>
     <collision>
-      <origin xyz="0 0 0" rpy="0 0 ${pi}" />
+      <origin xyz="0 0 0.11485" rpy="0 0 ${pi}" />
       <geometry>
-	<mesh filename="package://hydra/models/gripper_placer/meshes/gripper_pad_v2.stl" scale="0.01 0.01 0.01" />
+	<mesh filename="package://hydra/models/gripper_placer/meshes/gripper_pad_v2.stl" scale="${stl_scale} ${stl_scale} ${stl_scale}" />
       </geometry>
     </collision>

Commit message: Added gazebo tags to gripper in hopes of resolving physics --- did not help

File: models/gripper_placer/gripper_placer.urdf.xacro (robot description, xacro)
@@ -127,3 +127,10 @@
     </transmission>
   </xacro:if>
+  <!-- Gazebo tag for hopefully changing physics engine properties to work -->
+  <gazebo>
+    <maxVel>0</maxVel>
+    <minDepth>0.0001</minDepth>
+    <mu1>1000</mu1>
+    <mu2>1000</mu2>
+  </gazebo>
 </robot>

File: models/hydra/hydra.urdf (robot description, URDF)
Before this commit: robot hydra, 21 links, 20 joints
Links:
- added link gripper_center, mass 0.01
- added link side_d, mass 0.001; collision mesh filename=package://hydra/models/gripper_placer/meshes/gripper_pad_v2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 scale=0.0254 0.0254 0.0254; visual mesh filename=package://hydra/models/gripper_placer/meshes/gripper_pad_v2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 scale=0.0254 0.0254 0.0254
- added link side_p, mass 0.001; collision mesh filename=package://hydra/models/gripper_placer/meshes/gripper_pad_v2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 scale=0.0254 0.0254 0.0254; visual mesh filename=package://hydra/models/gripper_placer/meshes/gripper_pad_v2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 scale=0.0254 0.0254 0.0254
Joints:
- added joint gripper_joint_d: type prismatic, parent gripper_center, child side_d, origin xyz=0 0 0 rpy=0 0 0, axis 0 1 0, limit lower=-100 upper=100 effort=5000 velocity=0.5
- added joint gripper_joint_p: type prismatic, parent gripper_center, child side_p, origin xyz=0 0 0 rpy=0 0 0, axis 0 1 0, limit lower=-100 upper=100 effort=5000 velocity=0.5
- added joint mount_gripper_to_placer: type fixed, parent placer_tool0, child gripper_center, origin xyz=0 0 0 rpy=0 0 0

Commit message: Trying different approaches to fix physics

File: models/gripper_placer/gripper_placer.urdf.xacro (robot description, xacro)
@@ -2,4 +2,15 @@
 <robot name="gripper_placer"
        xmlns:xacro="http://ros.org/wiki/xacro">
+  <xacro:arg name="with_gripper_instead_of_forks" default="false" />
+  <xacro:if value="$(arg with_gripper_instead_of_forks)">
+    <xacro:property name="tool_offset_z" value="0.11485" />
+    <xacro:property name="tool_rotation_z" value="0" />
+    <xacro:property name="tool_stl_path" value="package://hydra/models/gripper_placer/meshes/gripper_pad_v2.stl" />
+  </xacro:if>
+  <xacro:unless value="$(arg with_gripper_instead_of_forks)">
+    <xacro:property name="tool_offset_z" value="0" />
+    <xacro:property name="tool_rotation_z" value="${pi/2}" />
+    <xacro:property name="tool_stl_path" value="package://hydra/models/gripper_placer/meshes/forks.stl" />
+  </xacro:unless>
   <!-- Switch between EffortJointInterface and PositionJointInterface, still requires change in yaml files -->
   <xacro:property name="using_position_not_effort" value="true" />
@@ -21,116 +32,138 @@
   <link name="side_p" >
     <visual>
-      <origin xyz="0 0 0.11485" rpy="0 0 0" />
+      <origin xyz="0 0 ${tool_offset_z}" rpy="0 0 ${tool_rotation_z}" />
       <geometry>
-	<mesh filename="package://hydra/models/gripper_placer/meshes/gripper_pad_v2.stl" scale="${stl_scale} ${stl_scale} ${stl_scale}" />
+	<mesh filename="${tool_stl_path}" scale="${stl_scale} ${stl_scale} ${stl_scale}" />
       </geometry>
     </visual>
     <collision>
-      <origin xyz="0 0 0.11485" rpy="0 0 0" />
+      <origin xyz="0 0 ${tool_offset_z}" rpy="0 0 ${tool_rotation_z}" />
       <geometry>
-	<mesh filename="package://hydra/models/gripper_placer/meshes/gripper_pad_v2.stl" scale="${stl_scale} ${stl_scale} ${stl_scale}" />
+	<mesh filename="${tool_stl_path}" scale="${stl_scale} ${stl_scale} ${stl_scale}" />
       </geometry>
     </collision>
     <inertial>
-      <mass value="0.001" />
+      <mass value="0.01" />
       <inertia ixx="0.01" ixy="0.0" ixz="0.0" iyy="0.02" iyz="0.0" izz="0.02" />
     </inertial>
   </link>
   <!-- Second side of gripper -->
-  <link name="side_d" >
-    <visual>
-      <origin xyz="0 0 0.11485" rpy="0 0 ${pi}" /><!--origin xyz="0 0.04185 0" rpy="0 0 ${pi}" /-->
-      <geometry>
-	<mesh filename="package://hydra/models/gripper_placer/meshes/gripper_pad_v2.stl" scale="${stl_scale} ${stl_scale} ${stl_scale}" />
-      </geometry>
-    </visual>
-    <collision>
-      <origin xyz="0 0 0.11485" rpy="0 0 ${pi}" />
-      <geometry>
-	<mesh filename="package://hydra/models/gripper_placer/meshes/gripper_pad_v2.stl" scale="${stl_scale} ${stl_scale} ${stl_scale}" />
-      </geometry>
-    </collision>
-    <inertial>
-      <mass value="0.001" />
-      <inertia ixx="0.01" ixy="0.0" ixz="0.0" iyy="0.02" iyz="0.0" izz="0.02" />
-    </inertial>
-  </link>
-  <!-- Prismatic joint -->
-  <joint name="gripper_joint_p" type="prismatic">
-    <origin xyz="0 0 0" rpy="0 0 0" />
-    <axis xyz="0 1 0" />
-    <parent link="gripper_center" />
-    <child link="side_p" />
-    <limit effort="${effort_limit}" lower="-100" upper="100" velocity="0.5"/>
-  </joint>
-  <joint name="gripper_joint_d" type="prismatic">
-    <origin xyz="0 0 0" rpy="0 0 0" />
-    <axis xyz="0 1 0" />
-    <parent link="gripper_center" />
-    <child link="side_d" />
-    <limit effort="${effort_limit}" lower="-100" upper="100" velocity="0.5"/>
-  </joint>
-  <!-- Prismatic joint -->
-  <!--joint name="gripper_joint_p" type="fixed">
-    <origin xyz="0 0 0" rpy="0 0 0" />
-    <parent link="gripper_center" />
-    <child link="side_p" />
-  </joint>
-  <joint name="gripper_joint_d" type="fixed">
-    <origin xyz="0 0 0" rpy="0 0 0" />
-    <parent link="gripper_center" />
-    <child link="side_d" />
-    </joint-->
+  <xacro:if value="$(arg with_gripper_instead_of_forks)">
+    <link name="side_d" >
+      <visual>
+	<origin xyz="0 0 ${tool_offset_z}" rpy="0 0 ${pi}" />
+	<geometry>
+	  <mesh filename="${tool_stl_path}" scale="${stl_scale} ${stl_scale} ${stl_scale}" />
+	</geometry>
+      </visual>
+      <collision>
+	<origin xyz="0 0 ${tool_offset_z}" rpy="0 0 ${pi}" />
+	<geometry>
+	  <mesh filename="${tool_stl_path}" scale="${stl_scale} ${stl_scale} ${stl_scale}" />
+	</geometry>
+      </collision>
+      <inertial>
+	<mass value="0.01" />
+	<inertia ixx="0.01" ixy="0.0" ixz="0.0" iyy="0.02" iyz="0.0" izz="0.02" />
+      </inertial>
+    </link>
+    <!-- Prismatic joint -->
+    <joint name="gripper_joint_p" type="prismatic">
+      <origin xyz="0 0 0" rpy="0 0 0" />
+      <axis xyz="0 1 0" />
+      <parent link="gripper_center" />
+      <child link="side_p" />
+      <limit effort="${effort_limit}" lower="-100" upper="100" velocity="0.5"/>
+    </joint>
+    <joint name="gripper_joint_d" type="prismatic">
+      <origin xyz="0 0 0" rpy="0 0 0" />
+      <axis xyz="0 1 0" />
+      <parent link="gripper_center" />
+      <child link="side_d" />
+      <limit effort="${effort_limit}" lower="-100" upper="100" velocity="0.5"/>
+    </joint>
+    <!-- Prismatic joint -->
+    <!--joint name="gripper_joint_p" type="fixed">
+	<origin xyz="0 0 0" rpy="0 0 0" />
+	<parent link="gripper_center" />
+	<child link="side_p" />
+	</joint>
+	<joint name="gripper_joint_d" type="fixed">
+	<origin xyz="0 0 0" rpy="0 0 0" />
+	<parent link="gripper_center" />
+	<child link="side_d" />
+	</joint-->
     <!-- Transmission for ROS control -->
-  <xacro:if value="${using_position_not_effort == 'true'}">
-    <transmission name="gripper_joint_transmission_p">
-      <type>transmission_interface/SimpleTransmission</type>
-      <joint name="gripper_joint_p">
-	<hardwareInterface>hardware_interface/PositionJointInterface</hardwareInterface>
-      </joint>
-      <actuator name="gripper_joint_motor_p">
-	<hardwareInterface>hardware_interface/PositionJointInterface</hardwareInterface>
-	<mechanicalReduction>1</mechanicalReduction>
-      </actuator>
-    </transmission>
-    <transmission name="gripper_joint_transmission_d">
-      <type>transmission_interface/SimpleTransmission</type>
-      <joint name="gripper_joint_d">
-	<hardwareInterface>hardware_interface/PositionJointInterface</hardwareInterface>
-      </joint>
-      <actuator name="gripper_joint_motor_d">
-	<hardwareInterface>hardware_interface/PositionJointInterface</hardwareInterface>
-	<mechanicalReduction>1</mechanicalReduction>
-      </actuator>
-    </transmission>
-  </xacro:if>
-  <xacro:if value="${using_position_not_effort == 'false'}">
-    <transmission name="gripper_joint_transmission_p">
-      <type>transmission_interface/SimpleTransmission</type>
-      <joint name="gripper_joint_p">
-	<hardwareInterface>hardware_interface/EffortJointInterface</hardwareInterface>
-      </joint>
-      <actuator name="gripper_joint_motor_p">
-	<hardwareInterface>hardware_interface/EffortJointInterface</hardwareInterface>
-	<mechanicalReduction>1</mechanicalReduction>
-      </actuator>
-    </transmission>
-    <transmission name="gripper_joint_transmission_d">
-      <type>transmission_interface/SimpleTransmission</type>
-      <joint name="gripper_joint_d">
-	<hardwareInterface>hardware_interface/EffortJointInterface</hardwareInterface>
-      </joint>
-      <actuator name="gripper_joint_motor_d">
-	<hardwareInterface>hardware_interface/EffortJointInterface</hardwareInterface>
-	<mechanicalReduction>1</mechanicalReduction>
-      </actuator>
-    </transmission>
-  </xacro:if>
+    <xacro:if value="${using_position_not_effort == 'true'}">
+      <transmission name="gripper_joint_transmission_p">
+	<type>transmission_interface/SimpleTransmission</type>
+	<joint name="gripper_joint_p">
+	  <hardwareInterface>hardware_interface/PositionJointInterface</hardwareInterface>
+	</joint>
+	<actuator name="gripper_joint_motor_p">
+	  <hardwareInterface>hardware_interface/PositionJointInterface</hardwareInterface>
+	  <mechanicalReduction>1</mechanicalReduction>
+	</actuator>
+      </transmission>
+      <transmission name="gripper_joint_transmission_d">
+	<type>transmission_interface/SimpleTransmission</type>
+	<joint name="gripper_joint_d">
+	  <hardwareInterface>hardware_interface/PositionJointInterface</hardwareInterface>
+	</joint>
+	<actuator name="gripper_joint_motor_d">
+	  <hardwareInterface>hardware_interface/PositionJointInterface</hardwareInterface>
+	  <mechanicalReduction>1</mechanicalReduction>
+	</actuator>
+      </transmission>
+    </xacro:if>  <!-- End if for using_position_not_effort -->
+    <xacro:if value="${using_position_not_effort == 'false'}">
+      <transmission name="gripper_joint_transmission_p">
+	<type>transmission_interface/SimpleTransmission</type>
+	<joint name="gripper_joint_p">
+	  <hardwareInterface>hardware_interface/EffortJointInterface</hardwareInterface>
+	</joint>
+	<actuator name="gripper_joint_motor_p">
+	  <hardwareInterface>hardware_interface/EffortJointInterface</hardwareInterface>
+	  <mechanicalReduction>1</mechanicalReduction>
+	</actuator>
+      </transmission>
+      <transmission name="gripper_joint_transmission_d">
+	<type>transmission_interface/SimpleTransmission</type>
+	<joint name="gripper_joint_d">
+	  <hardwareInterface>hardware_interface/EffortJointInterface</hardwareInterface>
+	</joint>
+	<actuator name="gripper_joint_motor_d">
+	  <hardwareInterface>hardware_interface/EffortJointInterface</hardwareInterface>
+	  <mechanicalReduction>1</mechanicalReduction>
+	</actuator>
+      </transmission>
+    </xacro:if>  <!-- End branch for !using_position_not_effort -->
+    <gazebo reference="side_d">
+      <kp>1e12</kp>
+      <kd>1.0</kd>
+      <maxVel>0.0</maxVel>
+      <minDepth>0.001</minDepth>
+      <mu1>1000</mu1>
+      <mu2>1000</mu2>
+      <fdir1>0.0 0.0 0.0</fdir1>
+    </gazebo>
+  </xacro:if>  <!-- End branch for with_gripper_instead_of_forks -->
   <!-- Gazebo tag for hopefully changing physics engine properties to work -->
-  <gazebo>
-    <maxVel>0</maxVel>
-    <minDepth>0.0001</minDepth>
+  <gazebo reference="side_p">
+    <kp>1e12</kp>
+    <kd>1.0</kd>
+    <maxVel>0.0</maxVel>
+    <minDepth>0.001</minDepth>
     <mu1>1000</mu1>
     <mu2>1000</mu2>
+    <fdir1>0.0 0.0 0.0</fdir1>
   </gazebo>
+  <xacro:unless value="$(arg with_gripper_instead_of_forks)">
+    <!-- Fixed joint for forks -->
+    <joint name="gripper_joint_p" type="fixed">
+      <origin xyz="0 0 0" rpy="0 0 0" />
+      <parent link="gripper_center" />
+      <child link="side_p" />
+    </joint>
+  </xacro:unless>
 </robot>
