Commit message: Finished simulation without Kinect

File: models/depth_camera_kinect/kinect_properties.urdf.xacro (robot description, xacro)
@@ -3,5 +3,5 @@
       name="kinect_xacro_properties">
   <!-- Translation and rotation of camera from its base link -->
-  <xacro:property name="cam_px" value="-0.12" />
+  <xacro:property name="cam_px" value="-0.075" />
   <xacro:property name="cam_py" value="0" />
   <xacro:property name="cam_pz" value="0.08" />

File: models/ee_and_nailer/ee_and_nailer.urdf.xacro (robot description, xacro)
@@ -58,4 +58,5 @@
       </geometry>
     </visual>
+    <!--
     <collision>
       <origin xyz="0 0 0" rpy="0 0 0" />
@@ -64,4 +65,5 @@
       </geometry>
     </collision>
+    -->
     <inertial>
       <mass value="0.1" />

File: models/gripper_placer/gripper_placer.urdf.xacro (robot description, xacro)
@@ -51,5 +51,5 @@
       <origin xyz="0 0 .15" rpy="0 0 ${pi}" />
       <geometry>
-	<box size=".05 .01 .07" />
+	<box size=".10 .01 .07" />
       </geometry>
     </xacro:unless>
@@ -83,4 +83,26 @@
     <xacro:inertial_values />
     </link>
+    <xacro:unless value="$(arg stl_collision)">
+      <link name="fake_block" >
+	<!--
+	<visual>
+	  <geometry>
+	    <box size=".14 .01 .07" />
+	  </geometry>
+	  </visual>
+	  -->
+	<collision>
+	  <geometry>
+	    <box size=".14 .01 .07" />
+	  </geometry>
+	</collision>
+	<xacro:inertial_values />
+      </link>
+      <joint name="fake_block_joint" type="fixed">
+	<origin xyz="0 0.005 .452" rpy="0 0 0" />
+	<parent link="side_d" />
+	<child link="fake_block" />
+      </joint>
+    </xacro:unless>
     <!-- Prismatic joint -->
     <joint name="gripper_joint_p" type="prismatic">

File: models/hydra/hydra.urdf (robot description, URDF)
Before this commit: robot hydra, 21 links, 20 joints
Links:
- added link camera_depth_frame, mass 0.001
- added link camera_depth_optical_frame, mass 0.001
- added link camera_link, mass 0.001; collision box size=0.07271 0.27794 0.073; visual mesh filename=package://hydra/models/depth_camera_kinect/meshes/kinect.dae
- added link camera_rgb_frame, mass 0.001
- added link camera_rgb_optical_frame, mass 0.001
- added link ee_base, mass 0.1; collision mesh filename=package://hydra/models/ee_and_nailer/meshes/gripper_nailer_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 scale=0.0254 0.0254 0.0254; visual mesh filename=package://hydra/models/ee_and_nailer/meshes/gripper_nailer_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 scale=0.0254 0.0254 0.0254
- added link ee_center, mass 0.01
- added link ee_cover, mass 0.1; collision mesh filename=package://hydra/models/ee_and_nailer/meshes/gripper_nailer_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 scale=0.0254 0.0254 0.0254; visual mesh filename=package://hydra/models/ee_and_nailer/meshes/gripper_nailer_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 scale=0.0254 0.0254 0.0254
- added link gripper_center, mass 0.01
- added link nailer, mass 0.1; collision mesh filename=package://hydra/models/ee_and_nailer/meshes/nailer.stl scale=0.0254 0.0254 0.0254; visual mesh filename=package://hydra/models/ee_and_nailer/meshes/nailer.stl scale=0.0254 0.0254 0.0254
- added link side_d, mass 0.1; collision box size=.05 .01 .07; visual box size=.05 .01 .07
- added link side_p, mass 0.1; collision box size=.05 .01 .07; visual box size=.05 .01 .07
Joints:
- added joint camera_depth_joint: type fixed, parent camera_rgb_frame, child camera_depth_frame, origin xyz=0 0 0 rpy=0 0 0
- added joint camera_depth_optical_joint: type fixed, parent camera_depth_frame, child camera_depth_optical_frame, origin xyz=0 0 0 rpy=-1.57079632679 0 -1.57079632679
- added joint camera_joint: type fixed, parent camera_rgb_frame, child camera_link, origin xyz=-0.031 0 -0.016 rpy=0 0 0
- added joint camera_rgb_joint: type fixed, parent attacher_tool0, child camera_rgb_frame, origin xyz=-0.12 0 0.08 rpy=0 -1.5708 0
- added joint camera_rgb_optical_joint: type fixed, parent camera_rgb_frame, child camera_rgb_optical_frame, origin xyz=0 0 0 rpy=-1.57079632679 0 -1.57079632679
- added joint ee_base_joint: type fixed, parent ee_center, child ee_base, origin xyz=0 0 0 rpy=0 0 0
- added joint ee_cover_joint: type fixed, parent ee_center, child ee_cover, origin xyz=-0.022 0 0.053 rpy=0 0 1.57079632679
- added joint gripper_joint_d: type prismatic, parent gripper_center, child side_d, origin xyz=0 -0.038 0 rpy=0 0 0, axis 0 1 0, limit lower=-100 upper=100 effort=100000 velocity=0.5
- added joint gripper_joint_p: type prismatic, parent gripper_center, child side_p, origin xyz=0 0.038 0 rpy=0 0 0, axis 0 1 0, limit lower=-100 upper=100 effort=100000 velocity=0.5
- added joint mount_gripper_to_placer: type fixed, parent placer_tool0, child gripper_center, origin xyz=0 0 0 rpy=0 0 0
- added joint mount_nailer_to_placer: type fixed, parent attacher_tool0, child ee_center, origin xyz=0 0 0 rpy=0 0 0
- added joint nailer_joint: type fixed, parent ee_center, child nailer, origin xyz=0.0 -0.09 0.085 rpy=0 -1.57079632679 3.14159265359
- joint attacher_world_joint: origin xyz=1.5 0.0 0.0 rpy=0.0 0.0 0.0 -> xyz=1.5 0.0 0.0 rpy=0.0 0.0 3.14159265359

File: models/hydra/hydra.urdf.xacro (robot description, xacro)
@@ -54,5 +54,5 @@
     <parent link="world" />
     <child link = "attacher_base_link" />
-    <origin xyz="1.5 0.0 0.0" rpy="0.0 0.0 0.0" />  <!-- This yaw value is just temporary for lab.  Revert to 0.0 afterward. -->
+    <origin xyz="1.5 0.0 0.0" rpy="0.0 0.0 ${pi}" />
   </joint>
   <xacro:if value="$(arg is_using_nailer)">
