Commit message: Finished simulation with Kinect.  Working on layout animation.

File: models/depth_camera_kinect/kinect.urdf.xacro (robot description, xacro)
@@ -39,4 +39,5 @@
 		</joint>
 		<link name="camera_link">
+			<!--
 			<visual>
 			 <origin xyz="0 0 0" rpy="0 0 ${M_PI/2}"/>
@@ -51,4 +52,5 @@
 				</geometry>
 			</collision>
+			-->
 			<inertial>
 				<mass value="0.001" />

File: models/hydra/hydra.urdf (robot description, URDF)
Before this commit: robot hydra, 33 links, 32 joints
Links:
- added link fake_block, mass 0.1; collision box size=.14 .01 .07
- link nailer: geometry visual mesh filename=package://hydra/models/ee_and_nailer/meshes/nailer.stl scale=0.0254 0.0254 0.0254
- link side_d: geometry collision box size=.10 .01 .07; visual box size=.10 .01 .07
- link side_p: geometry collision box size=.10 .01 .07; visual box size=.10 .01 .07
Joints:
- added joint fake_block_joint: type fixed, parent side_d, child fake_block, origin xyz=0 0.005 .452 rpy=0 0 0
- joint camera_rgb_joint: origin xyz=-0.12 0 0.08 rpy=0 -1.5708 0 -> xyz=-0.075 0 0.08 rpy=0 -1.5708 0
